File: MIDITheremin10-24.sch (EAGLE design)
At the start: 75 parts, among them IC1 TL072P, IC2 TL072P, Q1 2N3904, T1 2N3904, T2 2N3904, T3 2N3904, T4 2N3904, T5 2N3904

Commit message: These are updated Schematics
updated schematic and PCB
Parts:
- removed Q1: 2N3904, transistor-npn:2N3904
- removed U$1: LM2917, lm2917:LM2917
- added C25: 4.7uF, resistor:CPOL-USE2.5-7
- added C26: .1uF, resistor:C-EU050-025X075
- added C27: 1uF, resistor:CPOL-USE2.5-7
- added IND_1, IND_2, LM2917_1, LM2917_2, LM2917_3, LM2917_4, LM2917_5, LM2917_6, LM2917_7, LM2917_8, TP_FOUT, TP_GND, TP_LOSC, TP_LV+, TP_LV-, TP_POSC, TP_PV+, TP_PV-, VOUT, VOUT_GREF: (no value), pinhead:PINHD-1X1
- added J1: DCJ0202, con-jack:DCJ0202
- added R38: 10k, resistor:R-US_0411/3V
- added R39: 10, resistor:R-US_0411/3V
- added R40: 100, rcl:R-US_0411/3V
- added R41: 100k, pot:3RP/1610N
- added T6: 2N3904, transistor-neu-to92:2N3904
- C10, C11: device c-trimm:C-TRIMM3008 -> rcl:C-TRIMM3040.427
- C22: device resistor:C-EU050-025X075 -> resistor:CPOL-USE2.5-7
- C23: value 1uF -> 10uF; device resistor:C-EU050-025X075 -> resistor:CPOL-USE2.5-7
- C24: value 10uF -> .1uF
- R16: value Rfreq -> 10k
- R27: value 100k -> 56k
- R28: value 100k -> 33k
Connections:
- removed net N$29: Q1.C, R36.1
- removed net N$30: R33.2, R34.1, U$1.4
- removed net N$32: R31.1, R32.1, R33.1, R37.1
- new net N$27: IC2B.-IN, IC2B.OUT, R39.1
- new net N$36: C24.2, IC2B.+IN, R16.1, R38.2
- new net N$38: R40.1, VOUT.1
- new net NON_INVERT_OUT: LM2917_4.1, LM2917_7.1, R33.2, R34.1
- net GND: now also R29.A, R3.2, R39.2, R41.E, R7.2, TP_GND.1; no longer C24.1, R16.1, R29.E, R3.1, R7.1, U$1.8
- net LOCAL_RESONANCE: now also C11.A; no longer C10.A
- net L_OSC_V+: now also C11.E, TP_LV+.1; no longer C10.E
- net L_OSC_V-: now also TP_LV-.1
- net N$11: now also IC1B.-IN, IC1B.OUT, TP_POSC.1; no longer IC1A.-IN, IC1A.OUT
- net N$12: now also IC1A.-IN, IC1A.OUT, TP_LOSC.1; no longer IC1B.-IN, IC1B.OUT
- net N$13: now also IC1B.+IN; no longer IC1A.+IN
- net N$14: now also R15.2; no longer R15.1
- net N$15: now also IC1A.+IN; no longer IC1B.+IN
- net N$16: now also R8.1; no longer R8.2
- net N$18: now also C23.+, R15.1, TP_FOUT.1; no longer R15.2, R16.2
- net N$19: now also IND_1.1
- net N$2: now also R4.2; no longer R4.1
- net N$20: now also C21.1, LM2917_2.1; no longer U$1.2
- net N$28: now also T6.B; no longer Q1.B
- net N$3: now also R3.1; no longer R3.2
- net N$31: now also C22.+, LM2917_6.1, R35.2, R36.2; no longer C24.2, R35.1
- net N$33: now also C27.+, LM2917_3.1; no longer U$1.3
- net N$34: now also C23.-, LM2917_1.1; no longer U$1.1
- net N$35: now also T6.E; no longer Q1.E
- net N$4: now also C10.A, IND_2.1; no longer C11.A
- net N$5: now also R4.1; no longer R4.2
- net N$7: now also R8.2; no longer R8.1
- net N$8: now also R7.1; no longer R7.2
- net P_OSC_V+: now also C10.E, TP_PV+.1; no longer C11.E
- net P_OSC_V-: now also R17.2, TP_PV-.1; no longer R17.1
- net V+: now also C24.1, C25.+, C26.2, J1.1, LM2917_5.1, R16.2, R29.E, R35.1; no longer R35.2, U$1.5
- net V-: now also C21.2, C22.-, C25.-, C26.1, C27.-, J1.2, J1.3, LM2917_8.1, R17.1, R31.1, R32.1, R33.1, R37.1, R38.1, R41.A, VOUT_GREF.1; no longer R17.2, R29.A
- net VOUT: now also R36.1, R40.2, T6.C; no longer U$1.7
- net V_CONTROL: now also R41.S
Other:
- note added: "Output voltage: when referenced to the virtual ground ont he PCB. OUTPUT (-6VDC to -1VDC) when referenced to the negative rail of the supply voltage OUTPUT(0 to +5vDC)"
- note added: "This is a multi-purpose input. when the sensor is stand alone. the potentiometer is connected for tuning. When used with our MIDI Board, the voltage control goes where pin 2 of the Pot is connected"
- moved on the sheet: C10, C11, C16, C17, C18, C19, C21, C24, C8, C9, IC1A, IC1B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

Commit message: Add files via upload
Parts:
- removed IND_1, IND_2: (no value), pinhead:PINHD-1X1
- removed R34: 620k, rcl:R-US_0411/3V
- removed R36, R37: 10k, rcl:R-US_0411/3V
- removed T6: 2N3904, transistor-neu-to92:2N3904
- added C28, C29, C30, C31: tune, resistor:C-EU050-025X075
- added L4, L5, L6: 10mH, rcl:L-US6000-XXX-RC
- added TP_VCONT: (no value), pinhead:PINHD-1X1
- L1, L2: device resistor:L-US0207/2V -> rcl:L-US6000-XXX-RC
- L3: value 40mH *** -> 10mH; device resistor:L-US0207/2V -> rcl:L-US6000-XXX-RC
- R27: value 56k -> 51k
- R28: value 33k -> 22k
Connections:
- removed net VOUT: R36.1, R40.2, T6.C
- new net ANT: ANT1.1, L6.2
- net LOCAL_RESONANCE: now also C28.2, C29.2
- net L_OSC_V+: now also C28.1, C29.1
- net N$19: now also L5.1, L6.1; no longer ANT1.1, IND_1.1, L3.1
- net N$28: now also L3.1, L4.1; no longer R34.2, T6.B
- net N$31: no longer R36.2
- net N$35: now also L4.2, L5.2; no longer R37.2, T6.E
- net N$4: now also C30.2, C31.2; no longer IND_2.1
- net N$9: now also TP_VCONT.1
- net NON_INVERT_OUT: now also R40.2; no longer R34.1
- net P_OSC_V+: now also C30.1, C31.1
- net V-: no longer R37.1
Other:
- moved on the sheet: ANT1, C1, C10, C11, C2, L1, L2, L3, R1, R2, R3, R4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
