File: MIDITheremin.brd (EAGLE design)
At the start: 101.6 x 76.2 mm, 104 parts, among them IC1 TL072P, IC2 TL072P, J1 DCJ0202, T1 2N3904, T2 2N3904, T3 2N3904, T4 2N3904, T5 2N3904

Commit message: Add files via upload
Parts:
- removed J1: DCJ0202, con-jack:DCJ0202
- removed R41: 100k, pot:3RP/1610N
- removed VOUT_GREF: (no value), pinhead:1X01
- added U$1: MIDIJACK, adafruit:CP-2350
- moved TP_GND 21.8 mm to (62.9, 29.2)
- moved VOUT 21.6 mm to (73.7, 6.35)
- moved C25 7.73 mm to (83.2, 11.4)
Connections:
- removed net N$38: R40.1, VOUT.1
- new net VOUT: R40.1, U$1.1, VOUT.1
- net GND: now also U$1.PE, U$1.PE1, U$1.PE2, U$1.PE@; no longer R41.3
- net V+: now also U$1.3; no longer J1.1
- net V-: now also U$1.2; no longer J1.2, J1.3, R41.1, VOUT_GREF.1
- net V_CONTROL: now also U$1.5; no longer R41.2
Routing:
- net VOUT: track 0.00 -> 126.4 mm
- net N$38: track 81.0 -> 12.1 mm
- net V+: track 234.5 -> 295.7 mm
- net P_OSC_V+: track 49.1 -> 99.3 mm
- net N$4: track 50.3 -> 98.9 mm
- net V_CONTROL: track 21.8 -> 54.0 mm
- net LOCAL_RESONANCE: track 95.4 -> 125.1 mm
- net N$5: track 8.78 -> 36.5 mm
- net N$22: track 12.3 -> 36.5 mm
- net L_OSC_V+: track 59.1 -> 82.9 mm
- net N$42: track 0.00 -> 17.6 mm
- net N$44: track 0.00 -> 17.6 mm
- net N$43: track 0.00 -> 17.6 mm
- net L_OSC_V-: track 52.6 -> 64.7 mm
- net N$45: track 0.00 -> 9.57 mm
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